File: Tetris/sch/tetris.kicad_pcb (KiCad board)
At the start: 2 copper layers, 33 x 91.4 mm, 76 parts, among them J1 SWD, Q1 HL4953A, Q2 HL4953A, Q3 HL4953A, Q4 HL4953A, SW1 Boot, SW3 TSX101G100-250, SW4 Reset, U1 CH32V203C8T6, U10 ZX-QC66-6.5CJ, U11 MCP6001T-I/OT-TUDI, U2 STP16CP05TTR, U3 74HCT595D, U4 TLV70433DBVR, U5 SZ421288N/64, U6 SZ421288N/64, U7 LM1085-ADJ, U8 ZX-QC66-6.5CJ, U9 ZX-QC66-6.5CJ

Commit message: PCB routing in progress
Parts:
- moved R24 7.67 mm to (101.0, 74.3)
- moved R7 2.11 mm to (125.1, 64.1), turned to 90 degrees
- moved R8 2.01 mm to (125.1, 67.9)
- moved TP14 1.27 mm to (114.9, 69.2)
- moved TP9 1.27 mm to (114.9, 67.9)
- moved TP11 0.64 mm to (118.7, 54.6)
- moved TP12 0.64 mm to (120.0, 54.6)
- moved TP10 0.63 mm to (117.5, 54.6)
- moved TP13 0.63 mm to (121.3, 54.6)
- moved C7 0.25 mm to (110.9, 67.9)
- moved TP15 0.25 mm to (116.5, 67.9)
- moved TP7 0.25 mm to (113.4, 67.9)
- moved TP8 0.25 mm to (113.4, 69.2)
- moved R2 0.13 mm to (130.7, 51.4)
- turned C22 to 180 degrees
Connections:
- U1 pad 18: /LED/S1 -> /LED/S2
- U1 pad 19: /LED/S2 -> /LED/S1
Routing:
- net GND: track 0.00 -> 169.6 mm, vias 0 -> 10
- net +3V3: track 0.00 -> 112.0 mm, vias 0 -> 2
- net +5V: track 0.00 -> 65.7 mm, vias 0 -> 1
- net Net-(U1-NRST): track 0.00 -> 32.4 mm, vias 0 -> 2
- net Net-(J1-Pin_3): track 0.00 -> 20.7 mm
- net Net-(J1-Pin_4): track 0.00 -> 17.3 mm
- net /LED/DI-ROW: track 0.00 -> 14.1 mm, vias 0 -> 1
- net /LED/DI-COL: track 0.00 -> 14.0 mm, vias 0 -> 1
- net /LED/~{CS}: track 0.00 -> 13.5 mm, vias 0 -> 1
- net /LED/CLK-ROW: track 0.00 -> 13.4 mm, vias 0 -> 1
- net /LED/CLK-COL: track 0.00 -> 12.4 mm, vias 0 -> 1
- net /LED/~{OE}: track 0.00 -> 12.0 mm, vias 0 -> 1
- net /Btns/B8: track 0.00 -> 9.32 mm
- net /LED/PWM: track 0.00 -> 8.87 mm
- net Net-(U2-~{OUT0}): track 0.00 -> 8.70 mm
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- added copper zone on B.Cu, net GND
- added copper zone on F.Cu, net GND

Commit message: Tetris PCB route in progress
Parts:
- moved Q1 25.0 mm to (127.6, 85.7), turned to 0 degrees
- moved Q2 24.7 mm to (127.6, 80.0), turned to 0 degrees
- moved Q3 24.1 mm to (103.5, 79.4), turned to 180 degrees
- moved Q4 24.1 mm to (103.5, 85.1), turned to 180 degrees
- moved C20 23.0 mm to (124.5, 90.2), turned to -90 degrees
- moved C17 22.2 mm to (106.7, 75.6), turned to 0 degrees
- moved C18 22.2 mm to (106.7, 88.9), turned to 0 degrees
- moved C19 21.8 mm to (124.5, 76.2), turned to 180 degrees
- moved R24 18.5 mm to (119.4, 73.0)
- moved R14 13.7 mm to (121.9, 82.5), turned to 0 degrees
- moved R18 12.8 mm to (109.2, 83.2), turned to 180 degrees
- moved R15 12.7 mm to (121.9, 85.1), turned to 0 degrees
- moved R19 12.7 mm to (109.2, 85.1), turned to 180 degrees
- moved R20 12.7 mm to (109.2, 87.6), turned to 90 degrees
- moved R13 12.7 mm to (121.9, 80.0), turned to 0 degrees
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Connections:
- Q1 pad 5: Net-(U5-COL7) -> Net-(U5-COL4)
- Q1 pad 6: Net-(U5-COL7) -> Net-(U5-COL4)
- Q1 pad 7: Net-(U5-COL8) -> Net-(U5-COL6)
- Q1 pad 8: Net-(U5-COL8) -> Net-(U5-COL6)
- Q2 pad 5: Net-(U5-COL5) -> Net-(U5-COL7)
- Q2 pad 6: Net-(U5-COL5) -> Net-(U5-COL7)
- Q2 pad 7: Net-(U5-COL6) -> Net-(U5-COL8)
- Q2 pad 8: Net-(U5-COL6) -> Net-(U5-COL8)
- Q3 pad 5: Net-(U5-COL3) -> Net-(U5-COL5)
- Q3 pad 6: Net-(U5-COL3) -> Net-(U5-COL5)
- Q3 pad 7: Net-(U5-COL4) -> Net-(U5-COL3)
- Q3 pad 8: Net-(U5-COL4) -> Net-(U5-COL3)
- Q4 pad 5: Net-(U5-COL1) -> Net-(U5-COL2)
- Q4 pad 6: Net-(U5-COL1) -> Net-(U5-COL2)
- Q4 pad 7: Net-(U5-COL2) -> Net-(U5-COL1)
- Q4 pad 8: Net-(U5-COL2) -> Net-(U5-COL1)
- R13 pad 2: Net-(Q1A-G) -> Net-(Q2A-G)
- R14 pad 2: Net-(Q1B-G) -> Net-(Q2B-G)
- R15 pad 2: Net-(Q2A-G) -> Net-(Q1A-G)
- R16 pad 2: Net-(Q2B-G) -> Net-(Q3B-G)
- R17 pad 2: Net-(Q3A-G) -> Net-(Q1B-G)
- R18 pad 2: Net-(Q3B-G) -> Net-(Q3A-G)
- R19 pad 2: Net-(Q4A-G) -> Net-(Q4B-G)
- R20 pad 2: Net-(Q4B-G) -> Net-(Q4A-G)
- U1 pad 34: Net-(J1-Pin_4) -> Net-(J1-Pin_3)
- U1 pad 37: Net-(J1-Pin_3) -> Net-(J1-Pin_4)
Routing:
- net GND: track 169.6 -> 321.2 mm, vias 10 -> 18
- net +5V: track 65.7 -> 153.3 mm, vias 1 -> 5
- net /LED/LED-Pwr: track 0.00 -> 84.4 mm
- net /Btns/B4: track 4.10 -> 81.7 mm, vias 0 -> 1
- net /Btns/B3: track 3.59 -> 79.9 mm, vias 0 -> 1
- net /Btns/B2: track 5.59 -> 77.1 mm, vias 0 -> 1
- net /Btns/B1: track 6.92 -> 75.7 mm, vias 0 -> 1
- net /LED/PWM: track 8.87 -> 76.5 mm, vias 0 -> 2
- net Net-(U5-COL1): track 0.00 -> 58.5 mm
- net Net-(U5-COL6): track 0.00 -> 52.6 mm
- net Net-(U5-COL2): track 0.00 -> 52.0 mm
- net Net-(U5-COL5): track 0.00 -> 51.1 mm
- net Net-(U5-COL3): track 0.00 -> 51.0 mm
- net /Btns/B5: track 5.92 -> 56.7 mm, vias 0 -> 1
- net /Btns/B6: track 7.02 -> 57.4 mm, vias 0 -> 1
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
Commit message: PCB is ready
Parts:
- moved U10 22.9 mm to (127.0, 119.6)
- moved U8 22.9 mm to (127.0, 127.2)
- moved SW3 19.2 mm to (106.0, 123.2)
- moved R12 4.26 mm to (116.2, 95.2)
- moved U9 3.81 mm to (117.5, 127.2)
- moved C11 3.17 mm to (116.8, 119.4)
- moved C2 0.30 mm to (114.9, 70.5)
Connections:
- U1 pad 11: /Btns/B2 -> /Btns/B5
- U1 pad 12: /Btns/B3 -> /Btns/B4
- U1 pad 13: /Btns/B4 -> /Btns/B3
- U1 pad 14: /Btns/B5 -> /Btns/B7
- U1 pad 15: /Btns/B6 -> /Btns/B2
- U1 pad 16: /Btns/B7 -> /Btns/B6
Routing:
- net /LED/LED-Pwr: track 84.4 -> 125.5 mm, vias 0 -> 2
- net /Btns/B5: track 56.7 -> 89.9 mm
- net Net-(U11--IN): track 0.00 -> 26.5 mm
- net +5V: track 153.3 -> 179.5 mm, vias 5 -> 6
- net Net-(U2-~{OUT12}): track 18.0 -> 41.5 mm, vias 1 -> 2
- net Net-(U2-~{OUT14}): track 20.9 -> 41.3 mm, vias 1 -> 2
- net /Btns/B7: track 55.3 -> 73.8 mm
- net /Btns/B6: track 57.4 -> 75.1 mm
- net /Btns/B2: track 77.1 -> 93.6 mm
- net Net-(U2-~{OUT10}): track 15.3 -> 31.6 mm, vias 1 -> 2
- net Net-(U2-~{OUT9}): track 15.6 -> 31.9 mm
- net Net-(U2-~{OUT13}): track 19.0 -> 33.8 mm, vias 1 -> 2
- net Net-(U5-COL1): track 58.5 -> 72.1 mm, vias 0 -> 1
- net /Btns/B8: track 55.0 -> 68.5 mm
- net Net-(U2-~{OUT15}): track 26.2 -> 38.7 mm, vias 1 -> 2
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- added copper zone on In1.Cu, net +3V3
- added copper zone on B.Cu, net /LED/LED-Pwr
- added copper zone on In1.Cu, net GND
- added copper zone on In2.Cu, net GND
Other:
- board size 33 x 91.4 mm -> 33 x 91.7 mm
- copper layers 2 -> 4
- rule pad_to_mask_clearance: 0.05 -> 0
- board text added: "Boot"
- board text added: "Reset"
