File: LedFlash/ledflash2/ledflash.kicad_pcb (KiCad board)
At the start: 2 copper layers, 22.9 x 33.7 mm, 26 parts, among them J1 Conn_01x02_Pin, SW1 SW_Push, U1 SN74LVC1G14DBV, U2 74HC590A

Commit message: ladflash update
Parts:
- C2: footprint Capacitor_THT:CP_Radial_D5.0mm_P2.50mm -> easyeda2kicad:CAP-TH_BD4.0-P1.50-D0.8-FD
- C5: footprint Capacitor_THT:CP_Radial_D5.0mm_P2.50mm -> Capacitor_THT:CP_Radial_D6.3mm_P2.50mm
- moved C2 1.36 mm to (152.4, 83.8)
- moved C5 0.64 mm to (167.1, 88.3)
Routing:
- net GND: track 14.0 -> 17.7 mm, vias 17 -> 19
- net Net-(D2-Pad2): track 9.68 -> 10.9 mm
- net Net-(U2-CPC): track 20.0 -> 19.1 mm
- net Net-(C1-Pad1): track 29.3 -> 29.8 mm
Other:
- board text added: "CC CA"
