File: LedFlash/ledflash2/ledflash.kicad_pcb (KiCad board)
At the start: 2 copper layers, 22.9 x 33.7 mm, 26 parts, among them J1 Conn_01x02_Pin, SW1 SW_Push, U1 SN74LVC1G14DBV, U2 74HC590A

Commit message: Update LedFlash (capacitors footprints and LED symbol)
Parts:
- C3, C4: value 4nf -> 1.0
- R2: value R -> 5K6
- R3: value R -> 2K7
- R4: value R -> 1K3
- R5: value R -> 6K2
- R6: value R -> 3K3
- R7: value R -> 1K6
- R8: value R -> 560R
- R9: value R -> 270R
Changed lines of the file:
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@@
 			)
 		)
-		(property "Value" "R"
+		(property "Value" "6K2"
 			(at 0 1.43 90)
 			(layer "F.Fab")
@@
 			)
 		)
-		(property "Value" "R"
+		(property "Value" "560R"
 			(at 0 1.43 90)
 			(layer "F.Fab")
@@
 			)
 		)
+		(property ki_fp_filters "LED* LED_SMD:* LED_THT:*")
 		(sheetname "Root")
 		(sheetfile "ledflash.kicad_sch")
@@
 			(remove_unused_layers no)
 			(net 16 "/2r/o")
-			(pinfunction "1")
-			(pintype "unspecified")
+			(pinfunction "BA")
+			(pintype "passive")
 		)
 		(pad "2" thru_hole rect
@@
 			(remove_unused_layers no)
 			(net 17 "Net-(JP1-C)")
-			(pinfunction "+")
-			(pintype "unspecified")
+			(pinfunction "K")
+			(pintype "passive")
 		)
 		(pad "3" thru_hole oval
@@
 			(remove_unused_layers no)
 			(net 11 "/3r1/o1")
-			(pinfunction "3")
-			(pintype "unspecified")
+			(pinfunction "GA")
+			(pintype "passive")
 		)
 		(pad "4" thru_hole oval
@@
 			(remove_unused_layers no)
 			(net 4 "/3r/o1")
-			(pinfunction "4")
-			(pintype "unspecified")
+			(pinfunction "RA")
+			(pintype "passive")
 		)
 		(model "C:/Users/RomanKhvatov/Documents/Kicad/easyeda2kicad/easyeda2kicad.3dshapes/LED-TH_4P-BD5.8-P1.30-RGB.wrl"
@@
 			)
 		)
-		(property "Value" "R"
+		(property "Value" "270R"
 			(at 0 1.43 90)
 			(layer "F.Fab")
@@
 			)
 		)
-		(property "Value" "R"
+		(property "Value" "1K3"
 			(at 0 1.43 90)
 			(layer "F.Fab")
@@
 			)
 		)
-		(property "Value" "R"
+		(property "Value" "5K6"
 			(at 0 1.43 90)
 			(layer "F.Fab")
@@
 		(sheetname "Root")
 		(sheetfile "ledflash.kicad_sch")
-		(attr through_hole)
+		(attr through_hole dnp)
 		(fp_line
 			(start -0.61 -0.82)
@@
 		(sheetname "Root")
 		(sheetfile "ledflash.kicad_sch")
-		(attr through_hole)
+		(attr through_hole dnp)
 		(fp_line
 			(start -2.250241 -1.839)
@@
 			)
 		)
-		(property "Value" "R"
+		(property "Value" "3K3"
 			(at 0 1.43 90)
 			(layer "F.Fab")
@@
 			)
 		)
-		(property "Value" "R"
+		(property "Value" "2K7"
 			(at 0 1.43 90)
 			(layer "F.Fab")
@@
 			)
 		)
-		(property "Value" "R"
+		(property "Value" "1K6"
 			(at 0 1.43 90)
 			(layer "F.Fab")
@@
 			)
 		)
-		(property "Value" "4nf"
+		(property "Value" "1.0"
 			(at 0 -1.43 90)
 			(layer "B.Fab")
@@
 			)
 		)
-		(property "Value" "4nf"
+		(property "Value" "1.0"
 			(at 0 -1.43 0)
 			(layer "B.Fab")
