File: LedFlash/ledflash2/ledflash.kicad_sch (KiCad schematic)
At the start: 13 parts, among them J1 Conn_01x02_Pin, SW1 SW_Push, U1 SN74LVC1G14DBV, U2 74HC590A

Commit message: Update LedFlash (capacitors footprints and LED symbol)
Parts:
- C2: footprint Capacitor_THT:CP_Radial_D5.0mm_P2.50mm -> easyeda2kicad:CAP-TH_BD4.0-P1.50-D0.8-FD
- C5: footprint Capacitor_THT:CP_Radial_D5.0mm_P2.50mm -> Capacitor_THT:CP_Radial_D6.3mm_P2.50mm
- LED1: symbol easyeda2kicad:TJ-L5FYTXHTCYLCRGB-A5 -> Device:LED_BKGR
Changed lines of the file:
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@@
 	(wire
 		(pts
-			(xy 195.58 88.9) (xy 208.28 88.9)
+			(xy 195.58 88.9) (xy 210.82 88.9)
 		)
 		(stroke
@@
 	(wire
 		(pts
+			(xy 223.52 88.9) (xy 223.52 109.22)
+		)
+		(stroke
+			(width 0)
+			(type default)
+		)
+	)
+	(wire
+		(pts
+			(xy 208.28 99.06) (xy 208.28 93.98)
+		)
+		(stroke
+			(width 0)
+			(type default)
+		)
+	)
+	(wire
+		(pts
 			(xy 118.11 57.15) (xy 118.11 80.01)
 		)
@@
 	(wire
 		(pts
-			(xy 204.47 93.98) (xy 208.28 93.98)
-		)
-		(stroke
-			(width 0)
-			(type default)
-		)
-	)
-	(wire
-		(pts
 			(xy 101.6 57.15) (xy 118.11 57.15)
 		)
@@
 	(wire
 		(pts
+			(xy 208.28 93.98) (xy 210.82 93.98)
+		)
+		(stroke
+			(width 0)
+			(type default)
+		)
+	)
+	(wire
+		(pts
 			(xy 168.91 97.79) (xy 182.88 97.79)
 		)
@@
 	(wire
 		(pts
+			(xy 220.98 88.9) (xy 223.52 88.9)
+		)
+		(stroke
+			(width 0)
+			(type default)
+		)
+	)
+	(wire
+		(pts
 			(xy 44.45 80.01) (xy 46.99 80.01)
 		)
@@
 	(wire
 		(pts
+			(xy 208.28 83.82) (xy 210.82 83.82)
+		)
+		(stroke
+			(width 0)
+			(type default)
+		)
+	)
+	(wire
+		(pts
 			(xy 161.29 77.47) (xy 182.88 77.47)
 		)
@@
 	(wire
 		(pts
+			(xy 223.52 109.22) (xy 204.47 109.22)
+		)
+		(stroke
+			(width 0)
+			(type default)
+		)
+	)
+	(wire
+		(pts
 			(xy 66.04 80.01) (xy 76.2 80.01)
 		)
@@
 		(pts
 			(xy 156.21 124.46) (xy 153.67 124.46)
-		)
-		(stroke
-			(width 0)
-			(type default)
-		)
-	)
-	(wire
-		(pts
-			(xy 204.47 109.22) (xy 204.47 93.98)
 		)
 		(stroke
@@
 			)
 		)
-		(property "Footprint" "Capacitor_THT:CP_Radial_D5.0mm_P2.50mm"
+		(property "Footprint" "easyeda2kicad:CAP-TH_BD4.0-P1.50-D0.8-FD"
 			(at 77.1652 91.44 0)
 			(effects
@@
 	)
 	(symbol
-		(lib_id "easyeda2kicad:TJ-L5FYTXHTCYLCRGB-A5")
-		(at 213.36 91.44 270)
+		(lib_id "Device:LED_BKGR")
+		(at 215.9 88.9 0)
+		(mirror y)
 		(unit 1)
 		(exclude_from_sim no)
@@
 		(on_board yes)
 		(dnp no)
-		(fields_autoplaced yes)
 		(property "Reference" "LED1"
-			(at 217.17 90.1699 90)
-			(effects
-				(font
-					(size 1.27 1.27)
-				)
-				(justify left)
+			(at 215.9 101.6 0)
+			(effects
+				(font
+					(size 1.27 1.27)
+				)
 			)
 		)
 		(property "Value" "TJ-L5FYTXHTCYLCRGB-A5"
-			(at 217.17 92.7099 90)
-			(effects
-				(font
-					(size 1.27 1.27)
-				)
-				(justify left)
+			(at 226.568 86.868 90)
+			(effects
+				(font
+					(size 1.27 1.27)
+				)
 			)
 		)
 		(property "Footprint" "easyeda2kicad:LED-TH_4P-BD5.8-P1.30"
-			(at 200.66 91.44 0)
+			(at 215.9 101.6 0)
 			(effects
 				(font
@@
 		)
 		(property "Datasheet" "https://lcsc.com/product-detail/Others_TOGIALED-TJ-L5FYTXHTCYLCRGB-A5_C330749.html"
-			(at 198.12 91.44 0)
+			(at 215.9 104.14 0)
 			(effects
 				(font
@@
 		)
 		(property "Description" ""
-			(at 213.36 91.44 0)
+			(at 215.9 88.9 0)
 			(effects
 				(font
@@
 		)
 		(property "LCSC Part" "C330749"
-			(at 195.58 91.44 0)
+			(at 215.9 106.68 0)
 			(effects
 				(font
@@
 			)
 		)
-		(property "Footprint" "Capacitor_THT:CP_Radial_D5.0mm_P2.50mm"
+		(property "Footprint" "Capacitor_THT:CP_Radial_D6.3mm_P2.50mm"
 			(at 119.0752 120.65 0)
 			(effects
