File: LedFlash/ledflash2/3r.kicad_sch (KiCad schematic)
At the start: 5 parts

Commit message: Update LedFlash (capacitors footprints and LED symbol)
Parts:
- D3, D4: symbol Diode:BAT54C -> Diode:BAT54A
Changed lines of the file:
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@@
 	)
 	(symbol
-		(lib_id "Diode:BAT54C")
+		(lib_id "Diode:BAT54A")
 		(at 127 96.52 90)
 		(unit 1)
@@
 	)
 	(symbol
-		(lib_id "Diode:BAT54C")
+		(lib_name "BAT54A_1")
+		(lib_id "Diode:BAT54A")
 		(at 127 72.39 90)
 		(unit 1)

Commit message: Updated Value BAT54C to BAT54A
Parts:
- D3, D4: value BAT54C -> BAT54A
Changed lines of the file:
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@@
 			)
 		)
-		(property "Value" "BAT54C"
+		(property "Value" "BAT54A"
 			(at 124.46 97.7899 90)
 			(effects
@@
 			)
 		)
-		(property "Value" "BAT54C"
+		(property "Value" "BAT54A"
 			(at 124.46 73.6599 90)
 			(effects
