File: WPlant/sch/main-ext/main-ext.kicad_pcb (KiCad board)
At the start: 4 copper layers, 155 x 93 mm, 182 parts, among them J1 PROG/JTAG, J10 Ext, J11 HSensor, J12 HSensor, J13 HSensor, J14 HSensor, J15 HSensor, J16 HSensor, J17 HSensor, J18 WaterLevel, J2 Battery, J3 Balance, J4 DE9_Receptacle, J6 Conn_01x08_Pin, J9 Leak, M1 Motor_DC, Q1 FDS9926A, Q2 FDS9926A, Q3 FDS9926A, Q4 FDS9926A, Q6 Si2301, Q7 BC817, SW1 SW_Push, SW2 SW_Push, SW3 SW_Push, U1 SIWG917Y121MGABAR, U10 SP485EEN-L/TR, U11 TXU0102QDCURQ1, U12 CD74HCT4051M96, U13 CD74HCT4051M96, U14 SN74LVC1G14DBV, U2 AP64352SP-13, U3 AP64352SP-13, U4 AP64352SP-13, U6 AP2204R-5.0, U7 74HC594, U9 INA180A2, X1 SIT1552AI-JE-DCC-32.768D

Commit message: Update WP Sch (sheets titles, replaced wires by bus, update components values)
Parts:
- C30, C34, C35: value 0.1 -> 1.0
- C36: value ? -> 2.2
- R21, R22: value 100K -> 510
- R32, R33: value R -> 10K
- R35: value ? -> 2M
- R36: value 100K -> 10K5
- R37: value 100K -> 2K
- R39: value 100K -> 1K
- R40: value R -> 2M
- R44, R45, R46, R47, R48, R49: value R -> 1K
Connections:
- net Net-(U7-QB) renamed /Valves/V7
- net Net-(U7-QC) renamed /Valves/V6
- net Net-(U7-QD) renamed /Valves/V5
- net Net-(U7-QE) renamed /Valves/V4
- net Net-(U7-QF) renamed /Valves/V3
- net Net-(U7-QG) renamed /Valves/V2
- net Net-(U7-QH) renamed /Valves/V1
