File: Robot/csence.kicad_sch (KiCad schematic)
At the start: 6 parts, among them U12 INA180A2

Commit message: Started PCB roughting
Parts:
- renumbered C40 to C43, C41 to C44, R32 to R41, R32 to R42, R33 to R43, U12 to U13

Commit message: Updated PCB & Patterns for Robot
Other:
- company: (none) -> RoboWay
- title: (none) -> Current Sense
Changed lines of the file:
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@@
 	(generator_version "9.0")
 	(paper "A4")
+	(title_block
+		(title "Current Sense")
+		(company "RoboWay")
+	)
 	(junction
 		(at 168.91 71.12)
