File: Robot/5reg.kicad_sch (KiCad schematic)
At the start: 11 parts, among them U9 SY8366HQQC

Commit message: Updated Robot SCH
Parts:
- C24: value 220x16V -> 470x16V
- L1: value L -> CDRH127L125NP-4R7NC (4u7); MPN (none) -> C2835875
Changed lines of the file:
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@@
 			)
 		)
-		(property "Value" "220x16V"
+		(property "Value" "470x16V"
 			(at 97.79 82.1689 0)
 			(effects
@@
 		(on_board yes)
 		(dnp no)
-		(fields_autoplaced yes)
 		(property "Reference" "L1"
-			(at 118.11 81.28 90)
-			(effects
-				(font
-					(size 1.27 1.27)
-				)
-			)
-		)
-		(property "Value" "L"
-			(at 118.11 83.82 90)
+			(at 117.602 83.566 90)
+			(effects
+				(font
+					(size 1.27 1.27)
+				)
+			)
+		)
+		(property "Value" "CDRH127L125NP-4R7NC (4u7)"
+			(at 110.236 89.154 90)
 			(effects
 				(font
@@
 			(effects
 				(font
+					(size 1.27 1.27)
+				)
+				(hide yes)
+			)
+		)
+		(property "MPN" "C2835875"
+			(at 118.11 86.36 90)
+			(effects
+				(font

Commit message: Started PCB roughting
Parts:
- C25: renamed from C22; footprint (none) -> Capacitor_SMD:C_0603_1608Metric_Pad1.08x0.95mm_HandSolder
- C26: renamed from C21; footprint (none) -> Capacitor_SMD:C_1210_3225Metric_Pad1.33x2.70mm_HandSolder
- C27: renamed from C24; footprint (none) -> Capacitor_THT:CP_Radial_D8.0mm_P3.80mm
- C28: renamed from C20; footprint (none) -> Capacitor_SMD:C_0603_1608Metric_Pad1.08x0.95mm_HandSolder
- C29: renamed from C23; footprint (none) -> Capacitor_SMD:C_1210_3225Metric_Pad1.33x2.70mm_HandSolder
- C30: renamed from C19; footprint (none) -> Capacitor_SMD:C_0603_1608Metric_Pad1.08x0.95mm_HandSolder
- L1: footprint (none) -> easyeda2kicad:IND-SMD_L12.0-W12.0_CDRH127XX
- R32: renamed from R20; footprint (none) -> Resistor_SMD:R_0603_1608Metric_Pad0.98x0.95mm_HandSolder
- R33: renamed from R18; footprint (none) -> Resistor_SMD:R_0603_1608Metric_Pad0.98x0.95mm_HandSolder
- R34: renamed from R19; footprint (none) -> Resistor_SMD:R_0603_1608Metric_Pad0.98x0.95mm_HandSolder
- renumbered U9 to U10

Commit message: Updated PCB & Patterns for Robot
Other:
- company: (none) -> RoboWay
- title: (none) -> DC/DC
Changed lines of the file:
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@@
 	(generator_version "9.0")
 	(paper "A4")
+	(title_block
+		(title "DC/DC")
+		(company "RoboWay")
+	)
 	(junction
 		(at 132.08 93.98)

Commit message: Updated PCB for Robot
Connections:
- net GND: now also U10.3 (NC), U10.4 (NC)
- no-connect marks 3 -> 1
Changed lines of the file:
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@@
+	)
+	(junction
+		(at 134.62 88.9)
+		(diameter 0)
+		(color 0 0 0 0)
 	)
 	(junction
@@
 		(at 161.29 86.36)
 	)
-	(no_connect
-		(at 135.89 91.44)
-	)
-	(no_connect
-		(at 135.89 88.9)
-	)
 	(wire
 		(pts
@@
 	(wire
 		(pts
+			(xy 134.62 91.44) (xy 134.62 88.9)
+		)
+		(stroke
+			(width 0)
+			(type default)
+		)
+	)
+	(wire
+		(pts
 			(xy 161.29 93.98) (xy 165.1 93.98)
 		)
@@
 	(wire
 		(pts
+			(xy 134.62 88.9) (xy 135.89 88.9)
+		)
+		(stroke
+			(width 0)
+			(type default)
+		)
+	)
+	(wire
+		(pts
+			(xy 132.08 88.9) (xy 134.62 88.9)
+		)
+		(stroke
+			(width 0)
+			(type default)
+		)
+	)
+	(wire
+		(pts
 			(xy 205.74 67.31) (xy 205.74 64.77)
 		)
@@
 		(pts
 			(xy 106.68 93.98) (xy 109.22 93.98)
+		)
+		(stroke
+			(width 0)
+			(type default)
+		)
+	)
+	(wire
+		(pts
+			(xy 135.89 91.44) (xy 134.62 91.44)
 		)
 		(stroke
@@
 					(unit 1)
 				)
+			)
+		)
+	)
+	(symbol
+		(lib_id "power:GND")
+		(at 132.08 88.9 270)
+		(unit 1)
+		(exclude_from_sim no)
+		(in_bom yes)
+		(on_board yes)
+		(dnp no)
+		(property "Reference" "#PWR0112"
+			(at 125.73 88.9 0)
+			(effects
+				(font
+					(size 1.27 1.27)
+				)
+				(hide yes)
+			)
+		)
+		(property "Value" "GND"
+			(at 131.826 91.186 90)
+			(effects
+				(font
+					(size 1.27 1.27)
+				)
+				(justify right)
+			)
+		)
+		(property "Footprint" ""
+			(at 132.08 88.9 0)
+			(effects
+				(font
+					(size 1.27 1.27)
+				)
+				(hide yes)
+			)
+		)
+		(property "Datasheet" ""
+			(at 132.08 88.9 0)
+			(effects
+				(font
+					(size 1.27 1.27)
+				)
+				(hide yes)
+			)
+		)
+		(property "Description" "Power symbol creates a global label with name \"GND\" , ground"
+			(at 132.08 88.9 0)
+			(effects
+				(font
+					(size 1.27 1.27)
+				)
+				(hide yes)
+			)
+		)
+		(pin "1"
+		)
+		(instances
+			(project "Robot"
+				(path "/c5aa62e4-5f59-48a4-ae5d-57fc70429dc3/e9eb70e2-5ab4-43f7-8ba2-9f48573f337e/379d4900-8cb5-4ffc-a0e9-9f4d9fa9e1b4"
+					(reference "#PWR0113")
+					(unit 1)
+				)
+				(path "/c5aa62e4-5f59-48a4-ae5d-57fc70429dc3/e9eb70e2-5ab4-43f7-8ba2-9f48573f337e/396d8ecc-fd40-478c-8d76-0500de851d1b"
+					(reference "#PWR0114")
+					(unit 1)
+				)
+				(path "/c5aa62e4-5f59-48a4-ae5d-57fc70429dc3/e9eb70e2-5ab4-43f7-8ba2-9f48573f337e/729ab04e-4e5c-4cc5-bbb7-a84e7aeb8517"
+					(reference "#PWR0112")
+					(unit 1)
+				)
