File: Robot/Robot.kicad_pcb (KiCad board)
At the start: 2 copper layers, 130 x 156 mm, 172 parts, among them J1 Servo1, J10 Lidar, J11 Console, J12 M1, J13 M2, J14 M3, J15 M4, J16 Battery, J17 DE9_Receptacle, J18 Balance, J2 Servo2, J3 Servo3, J4 Servo4, J5 Servo5, J6 Servo6, J7 Servo7, J8 Beacon, J9 DLED, Q1 DMP3036SSD, Q2 Si2003, SW1 User, SW2 Pwr, U1 ADC128D818, U10 SY8366HQQC, U11 SY8366HQQC, U12 SY8366HQQC, U13 INA180A2, U14 INA180A2, U15 INA180A2, U16 INA180A2, U2 MaixCAM2, U3 DRV8845RHHR, U4 ICE40UP5K-SG48ITR, U5 74HCT245, U6 MCP4728, U7 NC7SZ175, U8 TLV70212DBVR, U9 TMI6050-33

Commit message: Updated PCB for Robot (routing in progress)
Parts:
- moved C16 30.8 mm to (121.5, 117.5), turned to 180 degrees
- moved C20 29.5 mm to (117.2, 116.8), turned to 180 degrees
- moved U8 25.3 mm to (121.5, 120.8), turned to 180 degrees
- moved C10 23.2 mm to (122.0, 139.1), turned to 90 degrees
- moved C15 22.4 mm to (102.3, 131.1), turned to 180 degrees
- moved C17 20.8 mm to (121.5, 123.9), turned to 180 degrees
- moved C22 20.2 mm to (112.8, 120.8), turned to 180 degrees
- moved C19 18.6 mm to (122.0, 135.3), turned to 90 degrees
- moved C2 17.5 mm to (107.2, 137.5), turned to 180 degrees
- moved C18 16.3 mm to (121.7, 128.7), turned to 180 degrees
- moved R31 15.7 mm to (106.2, 134.9), turned to 90 degrees
- moved C24 15.5 mm to (108.5, 126.7), turned to 180 degrees
- moved U9 14.2 mm to (112.8, 123.9), turned to 90 degrees
- moved C14 12.8 mm to (108.0, 134.9), turned to 90 degrees
- moved U4 9.69 mm to (115.1, 135.6), turned to 180 degrees
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Connections:
- C1 pad 2: +3.3V -> +3V3
- C10 pad 2: +3.3V -> +3V3
- C11 pad 2: +3.3V -> +3V3
- C12 pad 1: +3.3V -> +3V3
- C2 pad 1: +3.3V -> +3V3
- C8 pad 1: +3.3V -> +3V3
- D1 pad 2: +3.3V -> +3V3
- D2 pad 2: +3.3V -> +3V3
- D3 pad 2: +3.3V -> +3V3
- J1 pad 2: /Power/Pwr1 -> /Power/Pwr2
- J10 pad 5: +3.3V -> +3V3
- J11 pad 1: +3.3V -> +3V3
- J12 pad 2: +3.3V -> +3V3
- J13 pad 2: +3.3V -> +3V3
- J14 pad 2: +3.3V -> +3V3
- J15 pad 2: +3.3V -> +3V3
- J2 pad 2: /Power/Pwr1 -> /Power/Pwr2
- J3 pad 2: /Power/Pwr1 -> /Power/Pwr2
- J4 pad 2: /Power/Pwr2 -> /Power/Pwr1
- J5 pad 2: /Power/Pwr2 -> /Power/Pwr1
- J6 pad 2: /Power/Pwr2 -> /Power/Pwr1
- J7 pad 2: /Power/Pwr2 -> /Power/Pwr1
- J8 pad 1: +3.3V -> +3V3
- J9 pad 1: /Power/Pwr1 -> /Power/Pwr2
- R1 pad 1: +3.3V -> +3V3
- R11 pad 2: +3.3V -> +3V3
- R12 pad 2: +3.3V -> +3V3
- R13 pad 2: +3.3V -> +3V3
- R14 pad 2: +3.3V -> +3V3
- R15 pad 2: +3.3V -> +3V3
- R16 pad 2: +3.3V -> +3V3
- R17 pad 2: +3.3V -> +3V3
- R18 pad 2: +3.3V -> +3V3
- R2 pad 1: +3.3V -> +3V3
- R28 pad 2: +3.3V -> +3V3
- R29 pad 2: +3.3V -> +3V3
- R30 pad 2: +3.3V -> +3V3
- U1 pad 5: +3.3V -> +3V3
- U4 pad 1: +3.3V -> +3V3
- U4 pad 22: +3.3V -> +3V3
- U4 pad 33: +3.3V -> +3V3
- U6 pad 1: +3.3V -> +3V3
- U7 pad 3: +3.3V -> +3V3
- U7 pad 5: +3.3V -> +3V3
Routing:
- net +3V3: track 0.00 -> 620.5 mm, vias 0 -> 10
- net +3.3V: track 287.6 -> 0.00 mm, vias 2 -> 0
- net +5V: track 27.3 -> 279.8 mm, vias 4 -> 8
- net /Pots/Ref: track 0.00 -> 149.2 mm, vias 0 -> 2
- net /Power/Pwr2: track 35.1 -> 176.2 mm
- net /Pots/O1: track 0.00 -> 129.1 mm, vias 0 -> 2
- net /Pots/O2: track 0.00 -> 113.6 mm, vias 0 -> 2
- net +12V: track 97.9 -> 201.3 mm, vias 8 -> 11
- net /FPGA/SCL: track 0.00 -> 74.9 mm
- net /S5: track 3.53 -> 76.5 mm, vias 0 -> 2
- net /FPGA/SDA: track 0.00 -> 66.9 mm
- net /SP1: track 3.53 -> 62.6 mm, vias 0 -> 2
- net Net-(J14A-C1): track 3.27 -> 58.2 mm
- net Net-(J14A-C2): track 3.37 -> 57.0 mm
- net Net-(U3-I04): track 21.3 -> 73.3 mm
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