File: BigLED/draw/tpl.kicad_pcb (KiCad board)
At the start: 2 copper layers, 561.2 x 364 mm, 31 parts

Commit message: Added Wplant caps to BigLED acril cut drawing
Parts:
- added REF**: MountingHole_3.2mm_M3, MountingHole:MountingHole_3.2mm_M3, F.Cu at (132.3, 391.1)
- added REF**: MountingHole_3.2mm_M3, MountingHole:MountingHole_3.2mm_M3, F.Cu at (17.7, 405.9)
- added REF**1: MountingHole_3.2mm_M3, MountingHole:MountingHole_3.2mm_M3, F.Cu at (141.7, 405.9)
- added REF**2: MountingHole_3.2mm_M3, MountingHole:MountingHole_3.2mm_M3, F.Cu at (256.3, 391.1)
- added REF**3: MountingHole_3.2mm_M3, MountingHole:MountingHole_3.2mm_M3, F.Cu at (265.7, 405.9)
- added REF**4: MountingHole_3.2mm_M3, MountingHole:MountingHole_3.2mm_M3, F.Cu at (380.3, 391.1)
- added REF**5: MountingHole_3.2mm_M3, MountingHole:MountingHole_3.2mm_M3, F.Cu at (389.7, 405.9)
- added REF**6: MountingHole_3.2mm_M3, MountingHole:MountingHole_3.2mm_M3, F.Cu at (504.3, 391.1)
Other:
- board size 561.2 x 364 mm -> 561.2 x 407 mm
