File: WPlant/sch/but-ext-1/but1.kicad_sch (KiCad schematic)
At the start: 28 parts, among them J1 Conn_01x02_Pin, J4 But2, J8 MainModule, Q1 SI2301, Q2 Si2302, SW1 SW_Push, SW2 SW_Push, SW3 SW_Push, SW4 SW_Push, U1 TS3A44159PWR, U2 SMTSOM365BTR, U3 SMTSOM365BTR

Commit message: Added PCB templates for 2 boards around eInk display
Parts:
- removed D4, D5: BAT54C, Package_TO_SOT_SMD:SOT-23, symbol Diode:BAT54C
- removed H2: MountingHole, symbol Mechanical:MountingHole
- removed SW4: SW_Push, symbol Switch:SW_Push
- C1, C2: footprint (none) -> Capacitor_SMD:C_0603_1608Metric_Pad1.08x0.95mm_HandSolder
- C3: footprint (none) -> easyeda2kicad:CAP-TH_BD5.0-P2.00-D0.8-FD
- H1: footprint (none) -> MountingHole:MountingHole_3mm
- J1: footprint (none) -> Connector_JST:JST_XH_B2B-XH-A_1x02_P2.50mm_Vertical
- J4: footprint (none) -> Connector_PinHeader_2.54mm:PinHeader_2x06_P2.54mm_Vertical
- J8: footprint locals:CONN-TH_XAD-12AS -> but:CONN-TH_XAD-12AS
- R1, R2, R3, R4, R5, R6, R7, R8: footprint (none) -> Resistor_SMD:R_0603_1608Metric_Pad0.98x0.95mm_HandSolder
- SW1, SW2, SW3: footprint (none) -> Button_Switch_THT:SW_PUSH_6mm_H13mm

Commit message: Add 3D model of Robots head pole support
Parts:
- Q1: footprint easyeda2kicad:SOT-23-3_L3.0-W1.7-P0.95-LS2.9-BR -> Package_TO_SOT_SMD:SOT-23
- Q2: footprint easyeda2kicad:SOT-23_L2.9-W1.3-P1.90-LS2.4-BR -> Package_TO_SOT_SMD:SOT-23
- U2, U3: footprint easyeda2kicad:SMD_BD5.6-D4.1 -> but:SMD_BD5.6-D4.1
Changed lines of the file:
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@@
 			)
 		)
-		(property "Footprint" "easyeda2kicad:SMD_BD5.6-D4.1"
+		(property "Footprint" "but:SMD_BD5.6-D4.1"
 			(at 241.3 49.53 0)
 			(hide yes)
@@
 			)
 		)
-		(property "Footprint" "easyeda2kicad:SMD_BD5.6-D4.1"
+		(property "Footprint" "but:SMD_BD5.6-D4.1"
 			(at 241.3 41.91 0)
 			(hide yes)
@@
 			)
 		)
-		(property "Footprint" "easyeda2kicad:SOT-23_L2.9-W1.3-P1.90-LS2.4-BR"
+		(property "Footprint" "Package_TO_SOT_SMD:SOT-23"
 			(at 121.92 163.83 0)
 			(hide yes)
@@
 			)
 		)
-		(property "Footprint" "easyeda2kicad:SOT-23-3_L3.0-W1.7-P0.95-LS2.9-BR"
+		(property "Footprint" "Package_TO_SOT_SMD:SOT-23"
 			(at 111.76 130.81 0)
 			(hide yes)
