File: FPLock/sch-main/Power.kicad_sch (KiCad schematic)
At the start: 69 parts, among them J3 Cluch, Q1 AO4407A, Q2 IRLL2705TRPBF, Q3 SI2301CDS-T1-GE3, Q4 Si2302CDS-T1-GE3, Q5 Si2302CDS-T1-GE3, U10 FP6296XR-G1, U11 MS7208ABC, U12 AAT3221, U8 TMI6050-33, U9 IP2315

Commit message: Update I2C address
Parts:
- added JP2: SolderJumper_2_Open, Jumper:SolderJumper-2_P1.3mm_Open_RoundedPad1.0x1.5mm, symbol Jumper:SolderJumper_2_Open
- BT1: footprint (none) -> locals:Bat21700+
- C11, C17, C18, C21, C28, C29, C37, C38: footprint (none) -> locals:C_1210_3225Metric_Pad1.33x2.70mm_HandSolderExt
- C19, C40, C42, C43: footprint (none) -> easyeda2kicad:CAP-TH_BD6.3-P2.50-D0.6-FD-1
- C20, C22, C24, C25, C26, C27, C30, C33, C34, C35, C36: footprint (none) -> Capacitor_SMD:C_0603_1608Metric_Pad1.08x0.95mm_HandSolder
- C23, C39, C41: footprint Capacitor_SMD:C_1206_3216Metric_Pad1.33x1.80mm_HandSolder -> locals:C_1206_3216Metric_Pad1.33x1.80mm_HandSolderPlus
- D10: footprint Diode_THT:D_DO-35_SOD27_P7.62mm_Horizontal -> easyeda2kicad:LED0805-RD
- D4, D7: footprint (none) -> LED_THT:LED_D5.0mm
- D6, D8: footprint (none) -> Diode_SMD:D_SMC_Handsoldering
- D9: footprint (none) -> Diode_SMD:D_SMB_Handsoldering
- J3: footprint (none) -> Connector_PinHeader_2.54mm:PinHeader_1x02_P2.54mm_Vertical
- L3: footprint (none) -> easyeda2kicad:IND-SMD_L7.0-W6.9_APZBX0650M
- R31, R32, R33, R34, R35, R36, R37, R38, R39, R40, R41, R42, R43, R44, R45, R46, R47, R48, R49, R50: footprint (none) -> Resistor_SMD:R_0603_1608Metric_Pad0.98x0.95mm_HandSolder
Connections:
- net at C21.1, C22.1, C24.1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: now also JP2.2 (B); no longer BT1.1 (+)
- new net: BT1.1 (+), JP2.1 (A)
Other:
- moved on the sheet: BT1
