File: FPLock/sch-main/stepper.kicad_sch (KiCad schematic)
At the start: 21 parts, among them J2 StepMotor, U6 A3979SLPTR-T, U7 HXY6206I-2.5

Commit message: Update I2C address
Parts:
- C10, C46, C47: footprint (none) -> locals:C_1210_3225Metric_Pad1.33x2.70mm_HandSolderExt
- C12, C13, C14, C15, C16, C7, C8, C9: footprint (none) -> Capacitor_SMD:C_0603_1608Metric_Pad1.08x0.95mm_HandSolder
- J2: footprint (none) -> Connector_PinHeader_2.54mm:PinHeader_1x04_P2.54mm_Vertical
- JP1: footprint (none) -> Jumper:SolderJumper-3_P1.3mm_Open_RoundedPad1.0x1.5mm
- R24, R25: footprint (none) -> Resistor_SMD:R_2512_6332Metric_Pad1.40x3.35mm_HandSolder
- R26, R27, R28, R29: footprint (none) -> Resistor_SMD:R_0603_1608Metric_Pad0.98x0.95mm_HandSolder
Connections:
- net at U6.18 (OUT2B): now also J2.4 (Pin_4); no longer J2.2 (Pin_2)
- net at U6.25 (OUT1B): now also J2.2 (Pin_2); no longer J2.1 (Pin_1)
- net at U6.4 (OUT1A): now also J2.1 (Pin_1); no longer J2.4 (Pin_4)
Other:
- note added: "2B 2A 1B 1A"
- note removed: "1B 2B 2A 1A"
- moved on the sheet: C16, J2
Changed lines of the file:
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@@
 		)
 	)
-	(text "1B\n2B\n2A\n1A\n"
+	(text "2B\n2A\n1B\n1A\n"
 		(exclude_from_sim no)
 		(at 277.876 123.19 0)
@@
 	(wire
 		(pts
-			(xy 187.96 121.92) (xy 270.51 121.92)
-		)
-		(stroke
-			(width 0)
-			(type default)
-		)
-	)
-	(wire
-		(pts
 			(xy 176.53 91.44) (xy 173.99 91.44)
 		)
@@
 	(wire
 		(pts
-			(xy 266.7 119.38) (xy 270.51 119.38)
-		)
-		(stroke
-			(width 0)
-			(type default)
-		)
-	)
-	(wire
-		(pts
 			(xy 76.2 105.41) (xy 62.23 105.41)
 		)
@@
 	(wire
 		(pts
-			(xy 119.38 81.28) (xy 119.38 127)
+			(xy 120.65 81.28) (xy 120.65 127)
 		)
 		(stroke
@@
 	(wire
 		(pts
-			(xy 165.1 119.38) (xy 162.56 119.38)
+			(xy 236.22 73.66) (xy 233.68 73.66)
 		)
 		(stroke
@@
 	(wire
 		(pts
-			(xy 121.92 99.06) (xy 121.92 124.46)
+			(xy 123.19 99.06) (xy 123.19 121.92)
 		)
 		(stroke
@@
 	(wire
 		(pts
-			(xy 187.96 99.06) (xy 187.96 121.92)
+			(xy 187.96 99.06) (xy 187.96 119.38)
 		)
 		(stroke
@@
 	(wire
 		(pts
-			(xy 173.99 88.9) (xy 205.74 88.9)
+			(xy 266.7 124.46) (xy 270.51 124.46)
 		)
 		(stroke
@@
 	(wire
 		(pts
-			(xy 201.93 87.63) (xy 201.93 83.82)
+			(xy 173.99 88.9) (xy 205.74 88.9)
 		)
 		(stroke
@@
 	(wire
 		(pts
-			(xy 138.43 78.74) (xy 146.05 78.74)
+			(xy 201.93 87.63) (xy 201.93 83.82)
 		)
 		(stroke
@@
 	(wire
 		(pts
-			(xy 119.38 127) (xy 270.51 127)
+			(xy 138.43 78.74) (xy 146.05 78.74)
 		)
 		(stroke
@@
 	(wire
 		(pts
-			(xy 121.92 124.46) (xy 270.51 124.46)
+			(xy 120.65 127) (xy 270.51 127)
 		)
 		(stroke
@@
 	(wire
 		(pts
-			(xy 173.99 81.28) (xy 266.7 81.28)
+			(xy 123.19 121.92) (xy 270.51 121.92)
 		)
 		(stroke
@@
 	(wire
 		(pts
-			(xy 133.35 101.6) (xy 133.35 106.68)
+			(xy 173.99 81.28) (xy 266.7 81.28)
 		)
 		(stroke
@@
 	(wire
 		(pts
-			(xy 266.7 81.28) (xy 266.7 119.38)
+			(xy 133.35 101.6) (xy 133.35 106.68)
 		)
 		(stroke
@@
 	(wire
 		(pts
-			(xy 146.05 81.28) (xy 119.38 81.28)
+			(xy 146.05 81.28) (xy 120.65 81.28)
 		)
 		(stroke
@@
 	(wire
 		(pts
-			(xy 146.05 99.06) (xy 121.92 99.06)
+			(xy 146.05 99.06) (xy 123.19 99.06)
 		)
 		(stroke
@@
 	(wire
 		(pts
-			(xy 151.13 119.38) (xy 154.94 119.38)
+			(xy 222.25 73.66) (xy 226.06 73.66)
 		)
 		(stroke
@@
 	(wire
 		(pts
+			(xy 266.7 81.28) (xy 266.7 124.46)
+		)
+		(stroke
+			(width 0)
+			(type default)
+		)
+	)
+	(wire
+		(pts
 			(xy 90.17 104.14) (xy 90.17 107.95)
 		)
@@
 		)
 	)
+	(wire
+		(pts
+			(xy 187.96 119.38) (xy 270.51 119.38)
+		)
+		(stroke
+			(width 0)
+			(type default)
+		)
+	)
 	(hierarchical_label "Enable"
 		(shape input)
@@
 			)
 		)
-		(property "Footprint" ""
+		(property "Footprint" "Capacitor_SMD:C_0603_1608Metric_Pad1.08x0.95mm_HandSolder"
 			(at 89.8652 82.55 0)
 			(hide yes)
@@
 			)
 		)
-		(property "Footprint" ""
+		(property "Footprint" "Jumper:SolderJumper-3_P1.3mm_Open_RoundedPad1.0x1.5mm"
 			(at 111.76 74.93 0)
 			(hide yes)
@@
 			)
 		)
-		(property "Footprint" ""
+		(property "Footprint" "Capacitor_SMD:C_0603_1608Metric_Pad1.08x0.95mm_HandSolder"
 			(at 77.1652 102.87 0)
 			(hide yes)
@@
 			)
 		)
-		(property "Footprint" ""
+		(property "Footprint" "Capacitor_SMD:C_0603_1608Metric_Pad1.08x0.95mm_HandSolder"
 			(at 199.39 82.8548 0)
 			(hide yes)
@@
 			)
 		)
-		(property "Footprint" ""
+		(property "Footprint" "Capacitor_SMD:C_0603_1608Metric_Pad1.08x0.95mm_HandSolder"
 			(at 45.4152 102.87 0)
 			(hide yes)
@@
 	(symbol
 		(lib_id "power:+VSW")
-		(at 165.1 119.38 270)
+		(at 236.22 73.66 270)
 		(unit 1)
 		(body_style 1)
@@
 		(fields_autoplaced yes)
 		(property "Reference" "#PWR044"
-			(at 161.29 119.38 0)
+			(at 232.41 73.66 0)
 			(hide yes)
 			(show_name no)
@@
 		)
 		(property "Value" "+VSW"
-			(at 168.91 119.3799 90)
+			(at 240.03 73.6599 90)
 			(show_name no)
 			(do_not_autoplace no)
@@
 		)
 		(property "Footprint" ""
-			(at 165.1 119.38 0)
+			(at 236.22 73.66 0)
 			(hide yes)
 			(show_name no)
@@
 		)
 		(property "Datasheet" ""
-			(at 165.1 119.38 0)
+			(at 236.22 73.66 0)
 			(hide yes)
 			(show_name no)
@@
 		)
 		(property "Description" "Power symbol creates a global label with name \"+VSW\""
-			(at 165.1 119.38 0)
+			(at 236.22 73.66 0)
 			(hide yes)
 			(show_name no)
@@
 			)
 		)
-		(property "Footprint" ""
+		(property "Footprint" "Capacitor_SMD:C_0603_1608Metric_Pad1.08x0.95mm_HandSolder"
 			(at 199.39 93.0148 0)
 			(hide yes)
@@
 		(in_pos_files yes)
 		(dnp no)
-		(fields_autoplaced yes)
 		(property "Reference" "#PWR075"
 			(at 124.46 106.68 0)
@@
 		)
 		(property "Value" "GND"
-			(at 127 106.6799 90)
+			(at 132.08 109.982 90)
 			(show_name no)
 			(do_not_autoplace no)
@@
 			)
 		)
-		(property "Footprint" ""
+		(property "Footprint" "Resistor_SMD:R_0603_1608Metric_Pad0.98x0.95mm_HandSolder"
 			(at 111.252 100.33 90)
 			(hide yes)
@@
 	(symbol
 		(lib_id "power:GND")
-		(at 151.13 119.38 270)
+		(at 222.25 73.66 270)
 		(unit 1)
 		(body_style 1)
@@
 		(fields_autoplaced yes)
 		(property "Reference" "#PWR045"
-			(at 144.78 119.38 0)
+			(at 215.9 73.66 0)
 			(hide yes)
 			(show_name no)
@@
 		)
 		(property "Value" "GND"
-			(at 147.32 119.3799 90)
+			(at 218.44 73.6599 90)
 			(show_name no)
 			(do_not_autoplace no)
@@
 		)
 		(property "Footprint" ""
-			(at 151.13 119.38 0)
+			(at 222.25 73.66 0)
 			(hide yes)
 			(show_name no)
@@
 		)
 		(property "Datasheet" ""
-			(at 151.13 119.38 0)
+			(at 222.25 73.66 0)
 			(hide yes)
 			(show_name no)
@@
 		)
 		(property "Description" "Power symbol creates a global label with name \"GND\" , ground"
-			(at 151.13 119.38 0)
+			(at 222.25 73.66 0)
 			(hide yes)
 			(show_name no)
@@
 	(symbol
 		(lib_id "Device:C")
-		(at 158.75 119.38 90)
+		(at 229.87 73.66 90)
 		(unit 1)
 		(body_style 1)
@@
 		(fields_autoplaced yes)
 		(property "Reference" "C16"
-			(at 158.75 111.76 90)
+			(at 229.87 66.04 90)
 			(show_name no)
 			(do_not_autoplace no)
@@
 		)
 		(property "Value" "1.0"
-			(at 158.75 114.3 90)
+			(at 229.87 68.58 90)
 			(show_name no)
 			(do_not_autoplace no)
@@
 			)
 		)
-		(property "Footprint" ""
-			(at 162.56 118.4148 0)
+		(property "Footprint" "Capacitor_SMD:C_0603_1608Metric_Pad1.08x0.95mm_HandSolder"
+			(at 233.68 72.6948 0)
 			(hide yes)
 			(show_name no)
@@
 		)
 		(property "Datasheet" ""
-			(at 158.75 119.38 0)
+			(at 229.87 73.66 0)
 			(hide yes)
 			(show_name no)
@@
 		)
 		(property "Description" "Unpolarized capacitor"
-			(at 158.75 119.38 0)
+			(at 229.87 73.66 0)
 			(hide yes)
 			(show_name no)
@@
 			)
 		)
-		(property "Footprint" ""
+		(property "Footprint" "Resistor_SMD:R_2512_6332Metric_Pad1.40x3.35mm_HandSolder"
 			(at 139.7 108.458 90)
 			(hide yes)
@@
 			)
 		)
-		(property "Footprint" ""
+		(property "Footprint" "Resistor_SMD:R_0603_1608Metric_Pad0.98x0.95mm_HandSolder"
 			(at 79.248 78.74 90)
 			(hide yes)
@@
 			)
 		)
-		(property "Footprint" ""
+		(property "Footprint" "Resistor_SMD:R_0603_1608Metric_Pad0.98x0.95mm_HandSolder"
 			(at 88.392 100.33 90)
 			(hide yes)
@@
 			)
 		)
-		(property "Footprint" ""
+		(property "Footprint" "locals:C_1210_3225Metric_Pad1.33x2.70mm_HandSolderExt"
 			(at 220.6752 102.87 0)
 			(hide yes)
@@
 	(symbol
 		(lib_id "Connector:Conn_01x04_Pin")
-		(at 275.59 121.92 0)
-		(mirror y)
+		(at 275.59 124.46 180)
 		(unit 1)
 		(body_style 1)
@@
 		(dnp no)
 		(property "Reference" "J2"
-			(at 274.955 114.3 0)
+			(at 274.955 132.08 0)
 			(show_name no)
 			(do_not_autoplace no)
@@
 		)
 		(property "Value" "StepMotor"
-			(at 274.955 116.84 0)
+			(at 274.955 129.54 0)
 			(show_name no)
 			(do_not_autoplace no)
@@
 			)
 		)
-		(property "Footprint" ""
-			(at 275.59 121.92 0)
+		(property "Footprint" "Connector_PinHeader_2.54mm:PinHeader_1x04_P2.54mm_Vertical"
+			(at 275.59 124.46 0)
 			(hide yes)
 			(show_name no)
@@
 		)
 		(property "Datasheet" ""
-			(at 275.59 121.92 0)
+			(at 275.59 124.46 0)
 			(hide yes)
 			(show_name no)
@@
 		)
 		(property "Description" "Generic connector, single row, 01x04, script generated"
-			(at 275.59 121.92 0)
+			(at 275.59 124.46 0)
 			(hide yes)
 			(show_name no)
@@
 			)
 		)
-		(property "Footprint" ""
+		(property "Footprint" "Capacitor_SMD:C_0603_1608Metric_Pad1.08x0.95mm_HandSolder"
 			(at 100.6348 96.52 0)
 			(hide yes)
@@
 			)
 		)
-		(property "Footprint" ""
+		(property "Footprint" "locals:C_1210_3225Metric_Pad1.33x2.70mm_HandSolderExt"
 			(at 253.6952 102.87 0)
 			(hide yes)
@@
 			)
 		)
-		(property "Footprint" ""
+		(property "Footprint" "locals:C_1210_3225Metric_Pad1.33x2.70mm_HandSolderExt"
 			(at 237.1852 102.87 0)
 			(hide yes)
@@
 			)
 		)
-		(property "Footprint" ""
+		(property "Footprint" "Resistor_SMD:R_0603_1608Metric_Pad0.98x0.95mm_HandSolder"
 			(at 83.82 93.218 90)
 			(hide yes)
@@
 			)
 		)
-		(property "Footprint" ""
+		(property "Footprint" "Resistor_SMD:R_2512_6332Metric_Pad1.40x3.35mm_HandSolder"
 			(at 139.7 75.438 90)
 			(hide yes)
@@
 			)
 		)
-		(property "Footprint" ""
+		(property "Footprint" "Capacitor_SMD:C_0603_1608Metric_Pad1.08x0.95mm_HandSolder"
 			(at 213.36 87.9348 0)
 			(hide yes)
